File: spiderlily.kicad_sch (KiCad schematic)
At the start: 125 parts, among them J2 Conn_01x04_MountingPin, J3 Conn_01x05, SW1 MX_SW_HS, SW10 MX_SW_HS, SW11 MX_SW_HS, SW12 MX_SW_HS, SW13 MX_SW_HS, SW14 MX_SW_HS, SW15 MX_SW_HS, SW16 MX_SW_HS, SW17 MX_SW_HS, SW18 MX_SW_HS, SW19 MX_SW_HS, SW2 MX_SW_HS, SW20 MX_SW_HS, SW21 MX_SW_HS, SW22 MX_SW_HS, SW23 MX_SW_HS, SW24 MX_SW_HS, SW25 MX_SW_HS, SW26 MX_SW_HS, SW27 MX_SW_HS, SW28 MX_SW_HS, SW29 MX_SW_HS, SW3 MX_SW_HS, SW30 MX_SW_HS, SW31 MX_SW_HS, SW32 MX_SW_HS, SW33 MX_SW_HS, SW34 MX_SW_HS, SW35 MX_SW_HS, SW36 MX_SW_HS, SW37 MX_SW_HS, SW38 MX_SW_HS, SW39 MX_SW_HS, SW4 MX_SW_HS, SW40 MX_SW_HS, SW41 MX_SW_HS, SW42 MX_SW_HS, SW43 MX_SW_HS, SW44 MX_SW_HS, SW45 MX_SW_HS, SW46 MX_SW_HS, SW47 MX_SW_HS, SW48 Boot, SW49 RESET, SW5 MX_SW_HS, SW6 MX_SW_HS, SW7 MX_SW_HS, SW8 MX_SW_HS, SW9 MX_SW_HS, U1 XC6206PxxxMR, U3 RP2040, U4 W25Q128JVS, Y1 12MHz

Commit message: few changes
Parts:
- added U2: SRV05-4, PCM_marbastlib-various:SOT-23-6-routable, symbol PCM_marbastlib-various:SRV05-4
Connections:
- net +5V: now also U2.5 (VP)
- net D+: now also U2.1 (IO1)
- net D-: now also U2.6 (IO4)
- net GND: now also J2.MP (MountPin), U2.2 (VN)
- no-connect marks 15 -> 16
Other:
- note added: "ESD"
- moved on the sheet: C10, C11, C12, C13, C14, C15, C16, C3, C4, C5, C6, C7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

Commit message: parts list, minor changes, logo
Parts:
- C1, C2, C6, C9: LCSC (none) -> C52923
- C10, C11, C12, C13, C14, C15, C16, C5, C7: LCSC (none) -> C1525
- C3, C4: LCSC (none) -> C1555
- C8: LCSC (none) -> C15525
- D1, D10, D11, D12, D13, D14, D15, D16, D17, D18, D19, D2, D20, D21, D22, D23, D24, D25, D26, D27, D28, D29, D3, D30, D31, D32, D33, D34, D35, D36, D37, D38, D39, D4, D40, D41, D42, D43, D44, D45, D46, D47, D5, D6, D7, D8, D9: LCSC (none) -> C81598
- J2: LCSC (none) -> C3029343
- R3, R4, R5: LCSC (none) -> C25905
- R6, R7: LCSC (none) -> C11702
- R8, R9: LCSC (none) -> C25100
- SW1, SW10, SW11, SW12, SW13, SW14, SW15, SW16, SW17, SW18, SW19, SW2, SW20, SW21, SW22, SW23, SW24, SW25, SW26, SW27, SW28, SW29, SW3, SW30, SW31, SW32, SW33, SW34, SW35, SW36, SW37, SW38, SW39, SW4, SW40, SW41, SW42, SW43, SW44, SW45, SW46, SW47, SW5, SW6, SW7, SW8, SW9: LCSC (none) -> C41430893
- SW48, SW49: LCSC (none) -> C318884
- U1: LCSC (none) -> C5446
- U2: LCSC (none) -> C85364
- U3: LCSC (none) -> C2040
- U4: LCSC (none) -> C97521
- Y1: LCSC (none) -> C9002
Other:
- moved on the sheet: C1, C2, U1

Commit message: fixing UDB connection
Parts:
- J2: footprint Connector_Molex:Molex_Pico-EZmate_78171-0004_1x04-1MP_P1.20mm_Vertical -> Connector_JST:JST_SH_BM04B-SRSS-TB_1x04-1MP_P1.00mm_Vertical
Connections:
- net D+: now also U2.3 (IO2), U2.4 (IO3); no longer U2.1 (IO1)
- net D-: now also U2.1 (IO1)
- no-connect marks 16 -> 14
Changed lines of the file:
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@@
 	)
 	(no_connect
-		(at 130.81 44.45)
-	)
-	(no_connect
 		(at 275.59 62.23)
 	)
 	(no_connect
-		(at 130.81 39.37)
-	)
-	(no_connect
 		(at 275.59 67.31)
 	)
@@
 	(wire
 		(pts
+			(xy 130.81 44.45) (xy 132.08 44.45)
+		)
+		(stroke
+			(width 0)
+			(type default)
+		)
+	)
+	(wire
+		(pts
 			(xy 215.9 158.75) (xy 215.9 160.02)
 		)
@@
 	(wire
 		(pts
+			(xy 104.14 44.45) (xy 105.41 44.45)
+		)
+		(stroke
+			(width 0)
+			(type default)
+		)
+	)
+	(wire
+		(pts
 			(xy 189.23 158.75) (xy 189.23 160.02)
 		)
@@
 	(wire
 		(pts
+			(xy 130.81 39.37) (xy 132.08 39.37)
+		)
+		(stroke
+			(width 0)
+			(type default)
+		)
+	)
+	(wire
+		(pts
 			(xy 274.32 87.63) (xy 275.59 87.63)
 		)
@@
 	(wire
 		(pts
-			(xy 104.14 39.37) (xy 105.41 39.37)
-		)
-		(stroke
-			(width 0)
-			(type default)
-		)
-	)
-	(wire
-		(pts
 			(xy 260.35 147.32) (xy 269.24 147.32)
 		)
@@
 	(wire
 		(pts
-			(xy 104.14 44.45) (xy 105.41 44.45)
-		)
-		(stroke
-			(width 0)
-			(type default)
-		)
-	)
-	(wire
-		(pts
 			(xy 180.34 158.75) (xy 180.34 160.02)
 		)
@@
 	(wire
 		(pts
+			(xy 104.14 39.37) (xy 105.41 39.37)
+		)
+		(stroke
+			(width 0)
+			(type default)
+		)
+	)
+	(wire
+		(pts
 			(xy 198.12 140.97) (xy 198.12 142.24)
 		)
@@
 		)
 	)
+	(global_label "D+"
+		(shape input)
+		(at 132.08 39.37 0)
+		(fields_autoplaced yes)
+		(effects
+			(font
+				(size 1.27 1.27)
+			)
+			(justify left)
+		)
+		(property "Intersheetrefs" "${INTERSHEET_REFS}"
+			(at 137.9076 39.37 0)
+			(effects
+				(font
+					(size 1.27 1.27)
+				)
+				(justify left)
+				(hide yes)
+			)
+		)
+	)
 	(global_label "XTAL_IN"
 		(shape input)
@@
 		)
 	)
+	(global_label "D-"
+		(shape input)
+		(at 104.14 39.37 180)
+		(fields_autoplaced yes)
+		(effects
+			(font
+				(size 1.27 1.27)
+			)
+			(justify right)
+		)
+		(property "Intersheetrefs" "${INTERSHEET_REFS}"
+			(at 98.3124 39.37 0)
+			(effects
+				(font
+					(size 1.27 1.27)
+				)
+				(justify right)
+				(hide yes)
+			)
+		)
+	)
 	(global_label "row0"
 		(shape input)
@@
 	(global_label "D+"
 		(shape input)
-		(at 104.14 39.37 180)
+		(at 132.08 44.45 0)
 		(fields_autoplaced yes)
 		(effects
@@
 				(size 1.27 1.27)
 			)
-			(justify right)
+			(justify left)
 		)
 		(property "Intersheetrefs" "${INTERSHEET_REFS}"
-			(at 98.3124 39.37 0)
+			(at 137.9076 44.45 0)
 			(effects
 				(font
 					(size 1.27 1.27)
 				)
-				(justify right)
+				(justify left)
 				(hide yes)
 			)
@@
 			)
 		)
-		(property "Footprint" "Connector_Molex:Molex_Pico-EZmate_78171-0004_1x04-1MP_P1.20mm_Vertical"
+		(property "Footprint" "Connector_JST:JST_SH_BM04B-SRSS-TB_1x04-1MP_P1.00mm_Vertical"
 			(at 172.72 83.82 0)
 			(effects

Commit message: updated ezmate to jst sh, fixed oritentation and clearence issues
Parts:
- J2: footprint Connector_JST:JST_SH_BM04B-SRSS-TB_1x04-1MP_P1.00mm_Vertical -> Connector_JST:JST_SH_SM04B-SRSS-TB_1x04-1MP_P1.00mm_Horizontal
Changed lines of the file:
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@@
 			)
 		)
-		(property "Footprint" "Connector_JST:JST_SH_BM04B-SRSS-TB_1x04-1MP_P1.00mm_Vertical"
+		(property "Footprint" "Connector_JST:JST_SH_SM04B-SRSS-TB_1x04-1MP_P1.00mm_Horizontal"
 			(at 172.72 83.82 0)
 			(effects
