File: spiderlily.kicad_pcb (KiCad board)
At the start: 2 copper layers, 241.3 x 74.6 mm, 126 parts, among them J2 Conn_01x04_MountingPin, J3 Conn_01x05, SW1 MX_SW_HS, SW10 MX_SW_HS, SW11 MX_SW_HS, SW12 MX_SW_HS, SW13 MX_SW_HS, SW14 MX_SW_HS, SW15 MX_SW_HS, SW16 MX_SW_HS, SW17 MX_SW_HS, SW18 MX_SW_HS, SW19 MX_SW_HS, SW2 MX_SW_HS, SW20 MX_SW_HS, SW21 MX_SW_HS, SW22 MX_SW_HS, SW23 MX_SW_HS, SW24 MX_SW_HS, SW25 MX_SW_HS, SW26 MX_SW_HS, SW27 MX_SW_HS, SW28 MX_SW_HS, SW29 MX_SW_HS, SW3 MX_SW_HS, SW30 MX_SW_HS, SW31 MX_SW_HS, SW32 MX_SW_HS, SW33 MX_SW_HS, SW34 MX_SW_HS, SW35 MX_SW_HS, SW36 MX_SW_HS, SW37 MX_SW_HS, SW38 MX_SW_HS, SW39 MX_SW_HS, SW4 MX_SW_HS, SW40 MX_SW_HS, SW41 MX_SW_HS, SW42 MX_SW_HS, SW43 MX_SW_HS, SW44 MX_SW_HS, SW45 MX_SW_HS, SW46 MX_SW_HS, SW47 MX_SW_HS, SW48 Boot, SW49 RESET, SW5 MX_SW_HS, SW6 MX_SW_HS, SW7 MX_SW_HS, SW8 MX_SW_HS, SW9 MX_SW_HS, U1 XC6206PxxxMR, U2 SRV05-4, U3 RP2040, U4 W25Q128JVS, Y1 12MHz

Commit message: added GND vias liberally
Parts:
- moved SW48 2.22 mm to (145.8, 50.2)
- moved R4 2.22 mm to (140.2, 49.6)
- moved R6 2.22 mm to (140.2, 52.2)
- moved R5 2.22 mm to (140.2, 50.8)
- moved C2 1.77 mm to (109.2, 69.1)
- moved C1 1.77 mm to (103.8, 67.5)
- moved U1 1.77 mm to (106.1, 69.9)
- moved C8 1.02 mm to (111.8, 67.2)
Routing:
- net GND: track 108.8 -> 98.8 mm, vias 30 -> 52
- net col6: track 109.4 -> 113.3 mm
- net +3V3: track 158.6 -> 156.3 mm
- net CS: track 60.9 -> 59.0 mm
- net D-: track 39.2 -> 40.1 mm
- net D+: track 39.9 -> 40.8 mm
